File: ecad/usb_sensor_module/usb_sensor_module.kicad_pcb (KiCad board)
At the start: 2 copper layers, 22.9 x 50.8 mm, 23 parts, among them J1 218-508, J2 218-504/000-604, U1 TLV61046ADB

Commit message: USB sensor module schematic & pcb update WIP
Parts:
- added D2: 1N5817, Diode_THT:D_DO-41_SOD81_P7.62mm_Horizontal, F.Cu at (30.5, 55.9)
Connections:
- C1 pad 1: USB -> Net-(D1-K)
- D1 pad 1: USB -> Net-(D1-K)
- L1 pad 1: USB -> Net-(D1-K)
- U1 pad 4: USB -> Net-(D1-K)
- U1 pad 6: USB -> Net-(D1-K)
Routing:
- net USB: track 31.4 -> 0.00 mm
