File: ecad/usb_sensor_module/usb_sensor_module.kicad_sch (KiCad schematic)
At the start: 19 parts, among them J1 218-508, J2 218-504/000-604, U1 TLV61046ADB

Commit message: USB sensor module schematic & pcb update WIP
Parts:
- removed J1: 218-508, ul_218-508_footprint:ul_218-508, symbol ul_218-508:218-508
- removed J2: 218-504/000-604, ul_218-504-000-604_footprint:ul_218-504-000-604, symbol ul_218-504-000-604:218-504_000-604
- added D2: 1N5817, Diode_THT:D_DO-41_SOD81_P7.62mm_Horizontal, symbol Diode:1N5817
- added J1: Screw_Terminal_01x04, symbol Connector:Screw_Terminal_01x04
- added J2: Screw_Terminal_01x08, symbol Connector:Screw_Terminal_01x08
Connections:
- net 24V: now also J1.1 (Pin_1), J1.3 (Pin_3)
- net A2: now also J2.8 (Pin_8)
- net A3: now also J2.6 (Pin_6)
- net A4: now also J2.4 (Pin_4)
- net A5: now also J2.2 (Pin_2)
- net GND: now also J2.1 (Pin_1), J2.3 (Pin_3), J2.5 (Pin_5), J2.7 (Pin_7)
- net USB: now also D2.2 (A); no longer C1.1, D1.1 (K), L1.1, U1.4 (EN), U1.6 (VI)
- net at R8.1: now also J1.2 (Pin_2)
- net at R9.1: now also J1.4 (Pin_4)
- new net: C1.1, D1.1 (K), D2.1 (K), L1.1, U1.4 (EN), U1.6 (VI)
Other:
- moved on the sheet: A1, D1, R1, R10, R2, R3, R4, R7, R8, R9
